File: Hardware/nRF9160 Thing Plus.sch (EAGLE design)
At the start: 89 parts, among them J1 USB Female C, J10 QWIIC_RIGHT_ANGLE, J2 CON-HEADER-1X12-MALE-PIN, J3 CON-HEADER-1X16-MALE-PIN, J4 CON-1909763-1, J6 CON-SIM-104224-0820, J7 CON-1909763-1, J8 CON-FTSH-105-XX-X-DV, Q1 MOSFET-P-SC89, Q2 MOSFET-DUAL-COMP-SOT563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

Commit message: Panel Fix
Issues spotted:
- USB-C connector was a two layer part instead of four. This caused an issue where the inner 3.3V copper layer was shorting to the ground layers on other layers through the USB support tabs.
- Running the panelizer tool cause Eagle to crash.

Changes Made:
- Replaced USB-C connector with 4-layer footprint varient
- Not sure what was causing Eagle to crash, but rotating the board 90 degrees fixed it
- Silk on the bottom layer wasn't orientated correctly after rotating the board. Checking the "spin" box on the silk flipped the silk like it should be for "Designed by", "X", "Y", and "Z" labels

Updated panel and gerbers with changes outlined above.
Parts:
- J1: device SparkFun-Connectors:USB_C_2-LAYER_PADS -> SparkFun-Connectors:USB_C_4-LAYER_PADS
Changed lines of the file:
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@@
 <part name="GND39" library="supply1" library_urn="urn:adsk.eagle:library:371" deviceset="GND" device=""/>
 <part name="+3V12" library="supply1" library_urn="urn:adsk.eagle:library:371" deviceset="+3V3" device=""/>
-<part name="J1" library="SparkFun-Connectors" deviceset="USB_C" device="_2-LAYER_PADS" value="USB Female C"/>
+<part name="J1" library="SparkFun-Connectors" deviceset="USB_C" device="_4-LAYER_PADS" value="USB Female C"/>
 <part name="R20" library="SparkFun-Resistors" deviceset="5.1KOHM" device="-0402T-1/16W-1%" value="5.1k"/>
 <part name="R21" library="SparkFun-Resistors" deviceset="5.1KOHM" device="-0402T-1/16W-1%" value="5.1k"/>
